File: einkScreen_PCB/einkScreen.kicad_pcb (KiCad board)
At the start: 2 copper layers, 100 x 83.4 mm, 75 parts, among them J1 GPIOS, J2 ICSP, J3 FH34SRJ-24S-0.5SH_50_, Q1 BSS138LT1G, Q2 BSS84LT1G, SW1 SW_Push, SW2 SW_Push, U1 ATmega328P-A, U2 ST25DV64K-JFR6D3, U3 TPS3839G25, U4 LD39050PUR, U5 TPS3839G33, Y2 X322516MOB4SI

Commit message: working BLE
Parts:
- removed 3V3, GND1, SCL1, SDA1, TP6, TP7, VCC1: TestPoint, TestPoint:TestPoint_Pad_2.5x2.5mm
- removed AE1: Antenna_Loop, PCB Coils:COIL_GENERATOR
- removed C1: 0.1F, Ironies_Libs:SuperCapacitor
- removed C10, C11, C14, C15, C2, C3, C4, C5, C6, C7, C8: 1uF, Capacitor_SMD:C_0805_2012Metric
- removed C12, C20, C25: 10uF, Capacitor_SMD:C_0805_2012Metric
- removed C13: 4.7uF, Capacitor_SMD:C_0805_2012Metric
- removed C16, C17: 22pF, Capacitor_SMD:C_0805_2012Metric
- removed C21: 10nF, Capacitor_SMD:C_0805_2012Metric
- removed C22, C23, C24: NC, Capacitor_SMD:C_0805_2012Metric_Pad1.18x1.45mm_HandSolder
- removed C9: 100nF, Capacitor_SMD:C_0805_2012Metric
- removed D1, D2, D3: MBR0530, Diode_SMD:D_SOD-123
- removed D4: LED, LED_SMD:LED_0805_2012Metric
- removed D5: RB520CS30L, Diode_SMD:D_SOD-882
- removed H1, H2: MountingHole, MountingHole:MountingHole_2.2mm_M2
- removed J1: GPIOS, Connector_PinHeader_2.54mm:PinHeader_1x02_P2.54mm_Vertical
- removed J2: ICSP, Connector_PinHeader_2.54mm:PinHeader_2x03_P2.54mm_Vertical
- removed J3: FH34SRJ-24S-0.5SH_50_, FH34SRJ-24S-0.5SH_50_:HRS_FH34SRJ-24S-0.5SH_50_
- removed JP1: BS, Jumper:SolderJumper-3_P1.3mm_Open_RoundedPad1.0x1.5mm_NumberLabels
- removed JP2: Power, Jumper:SolderJumper-3_P1.3mm_Open_RoundedPad1.0x1.5mm_NumberLabels
- removed L1: 68uH, Inductor_SMD:L_1210_3225Metric
- removed Q1: BSS138LT1G, Package_TO_SOT_SMD:SOT-23-3
- removed Q2: BSS84LT1G, Package_TO_SOT_SMD:SOT-23-3
- removed R1, R2, R3, R9: 10K, Resistor_SMD:R_0805_2012Metric
- removed R10, R12, R13, R14, R18, R7, R8: 0R, Resistor_SMD:R_0805_2012Metric_Pad1.20x1.40mm_HandSolder
- removed R11: 330R, Resistor_SMD:R_0805_2012Metric
- removed R15: 330R, Resistor_SMD:R_0805_2012Metric_Pad1.20x1.40mm_HandSolder
- removed R16: 220k, Resistor_SMD:R_0805_2012Metric
- removed R17: NC, Resistor_SMD:R_0805_2012Metric_Pad1.20x1.40mm_HandSolder
- removed R19, R20: 10k, Resistor_SMD:R_0805_2012Metric
- removed R4: 3R, Resistor_SMD:R_0805_2012Metric
- removed R5: 15K, Resistor_SMD:R_0805_2012Metric
- removed R6: 47K, Resistor_SMD:R_0805_2012Metric
- removed SW1, SW2: SW_Push, Button_Switch_SMD:Panasonic_EVQPUL_EVQPUC
- removed TP8: MCU_RST, TestPoint:TestPoint_Pad_2.5x2.5mm
- removed U1: ATmega328P-A, Package_QFP:TQFP-32_7x7mm_P0.8mm
- removed U2: ST25DV64K-JFR6D3, Package_DFN_QFN:ST_UFDFPN-12-1EP_3x3mm_P0.5mm_EP1.4x2.55mm
- removed U3: TPS3839G25, Package_TO_SOT_SMD:SOT-23
- removed U4: LD39050PUR, LD39050PUR:SON95P300X300X100-7N
- removed U5: TPS3839G33, Package_TO_SOT_SMD:SOT-23
- removed Y2: X322516MOB4SI, Crystal:Crystal_SMD_SeikoEpson_TSX3225-4Pin_3.2x2.5mm
Routing:
- net +3V3: track 305.8 -> 0.00 mm, vias 8 -> 0
- net /SCL: track 122.3 -> 0.00 mm, vias 4 -> 0
- net /SDA: track 121.2 -> 0.00 mm, vias 2 -> 0
- net /ST25_LPD: track 96.2 -> 0.00 mm, vias 2 -> 0
- net VCC: track 95.1 -> 0.00 mm, vias 5 -> 0
- net GND: track 91.9 -> 0.00 mm, vias 53 -> 0
- net /ST25_GPO: track 87.8 -> 0.00 mm, vias 2 -> 0
- net /MCU_RST: track 56.2 -> 0.00 mm, vias 3 -> 0
- net /SCREEN_PREVGL: track 48.0 -> 0.00 mm, vias 2 -> 0
- net /MCU_SCK: track 47.8 -> 0.00 mm, vias 3 -> 0
- net /BUTTON2: track 45.4 -> 0.00 mm, vias 2 -> 0
- net /MCU_MOSI: track 43.6 -> 0.00 mm, vias 2 -> 0
- net /BUTTON1: track 40.5 -> 0.00 mm, vias 2 -> 0
- net /SCREEN_PREVGH: track 38.8 -> 0.00 mm, vias 2 -> 0
- net /SCREEN_BUSY: track 38.6 -> 0.00 mm, vias 2 -> 0
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- removed copper zone on B.Cu, net GND
- removed copper zone on F.Cu, net GND
Other:
- board outline removed
- board text removed: "Ver 1.0 Base Coil values: outer diameter=42mm N=13, L=4.8uH, w=0.535mm, s=0.558mm"
- board text removed: "pads x:±5 y:-30"

Commit message: working kinda
Parts:
- added AE1: Antenna_Loop, PCB Coils:WPT_COIL, F.Cu at (127.8, 101.1)
- added C1: 100nF, Capacitor_SMD:C_0805_2012Metric, F.Cu at (140.5, 137.1)
- added C10: 1uF, Capacitor_SMD:C_0805_2012Metric, F.Cu at (108.4, 132.0)
- added C11: 1uF, Capacitor_SMD:C_0805_2012Metric, F.Cu at (108.4, 129.5)
- added C12: 4.7uF, Capacitor_SMD:C_0805_2012Metric, F.Cu at (98.6, 137.1)
- added C13: 4.7uF, Capacitor_SMD:C_0805_2012Metric, F.Cu at (105.0, 142.2)
- added C14: 10uF, Capacitor_SMD:C_0805_2012Metric, F.Cu at (151.3, 73.0)
- added C15: 2.2nF, Capacitor_SMD:C_0805_2012Metric, F.Cu at (129.7, 65.3)
- added C16: 100nF, Capacitor_SMD:C_0805_2012Metric, F.Cu at (128.9, 54.6)
- added C17: 100nF, Capacitor_SMD:C_0805_2012Metric, F.Cu at (148.8, 73.0)
- added C18: 100nF, Capacitor_SMD:C_0805_2012Metric, F.Cu at (148.8, 68.8)
- added C19: 10uF, Capacitor_SMD:C_0805_2012Metric, F.Cu at (151.3, 68.8)
- added C2: 1uF, Capacitor_SMD:C_0805_2012Metric, F.Cu at (115.1, 139.6)
- added C20: 1uF, Capacitor_SMD:C_0805_2012Metric, F.Cu at (155.1, 78.0)
- added C21: 10nF, Capacitor_SMD:C_0805_2012Metric, F.Cu at (140.5, 63.7)
- added C22: 10nF, Capacitor_SMD:C_0805_2012Metric, F.Cu at (141.1, 53.3)
- added C23: 470nF, Capacitor_SMD:C_0805_2012Metric, F.Cu at (143.7, 63.7)
- added C24: 470nF, Capacitor_SMD:C_0805_2012Metric, F.Cu at (144.3, 53.1)
- added C25: 22nF, Capacitor_SMD:C_0805_2012Metric, F.Cu at (146.9, 63.7)
- added C26: 22nF, Capacitor_SMD:C_0805_2012Metric, F.Cu at (147.5, 53.1)
- added C27: 4.7uF, Capacitor_SMD:C_0805_2012Metric, F.Cu at (151.9, 49.4)
- added C28: 10uF, Capacitor_SMD:C_0805_2012Metric, F.Cu at (143.7, 68.5)
- added C29: 100nF, Capacitor_SMD:C_0805_2012Metric, F.Cu at (98.4, 58.3)
- added C3: 1uF, Capacitor_SMD:C_0805_2012Metric, F.Cu at (115.1, 137.1)
- added C30: 10uF, Capacitor_SMD:C_0805_2012Metric, F.Cu at (98.4, 54.6)
- added C31: 100nF, Capacitor_SMD:C_0805_2012Metric, F.Cu at (128.9, 58.4)
- added C32: 33nF, Capacitor_SMD:C_0805_2012Metric, F.Cu at (135.7, 59.8)
- added C33: 100nF, Capacitor_SMD:C_0805_2012Metric, F.Cu at (135.7, 62.8)
- added C34: 22nF, Capacitor_SMD:C_0805_2012Metric, F.Cu at (135.7, 65.8)
- added C4: 1uF, Capacitor_SMD:C_0805_2012Metric, F.Cu at (115.1, 134.5)
- added C5: 1uF, Capacitor_SMD:C_0805_2012Metric, F.Cu at (115.1, 132.0)
- added C6: 1uF, Capacitor_SMD:C_0805_2012Metric, F.Cu at (115.1, 129.5)
- added C7: 1uF, Capacitor_SMD:C_0805_2012Metric, F.Cu at (108.4, 139.6)
- added C8: 1uF, Capacitor_SMD:C_0805_2012Metric, F.Cu at (108.4, 137.1)
- added C9: 1uF, Capacitor_SMD:C_0805_2012Metric, F.Cu at (108.4, 134.5)
- added D1: MBR0530, Diode_SMD:D_SOD-123, F.Cu at (109.1, 144.1)
- added D2: MBR0530, Diode_SMD:D_SOD-123, F.Cu at (109.1, 147.2)
- added D3: MBR0530, Diode_SMD:D_SOD-123, F.Cu at (109.1, 150.4)
- added D4: LED, LED_SMD:LED_0805_2012Metric, F.Cu at (128.9, 52.1)
- added D5: 1N5819, Diode_SMD:D_SOD-123, F.Cu at (148.1, 139.6)
- added D6: ESD9B5.0ST5G, Diode_SMD:D_SOD-923, F.Cu at (145.6, 145.1)
- added D7: ESD9B5.0ST5G, Diode_SMD:D_SOD-923, F.Cu at (148.1, 145.1)
- added D8: ESD9B5.0ST5G, Diode_SMD:D_SOD-923, F.Cu at (150.7, 145.1)
- added J3: FH34SRJ-24S-0.5SH_50_, FH34SRJ-24S-0.5SH_50_:HRS_FH34SRJ-24S-0.5SH_50_, F.Cu at (128.0, 133.2)
- added J4: UART, Connector_PinSocket_2.54mm:PinSocket_1x04_P2.54mm_Vertical, F.Cu at (116.8, 72.4)
- added J5: 5VPWR, Connector_PinSocket_2.54mm:PinSocket_1x02_P2.54mm_Vertical, F.Cu at (155.8, 134.5)
- added JP1: BS, Jumper:SolderJumper-3_P1.3mm_Open_RoundedPad1.0x1.5mm_NumberLabels, F.Cu at (117.0, 142.2)
- added JP2: JumperEN, TestPoint:TestPoint_2Pads_Pitch2.54mm_Drill0.8mm, F.Cu at (134.6, 49.8)
- added JP3: RESE, Jumper:SolderJumper-3_P1.3mm_Open_RoundedPad1.0x1.5mm_NumberLabels, F.Cu at (100.5, 147.2)
- added JP4: JumperBOOT, TestPoint:TestPoint_2Pads_Pitch2.54mm_Drill0.8mm, F.Cu at (134.6, 53.6)
- added L1: 10uH, Inductor_SMD:L_1210_3225Metric, F.Cu at (103.0, 137.1)
- added Q1: A03400, Package_TO_SOT_SMD:TSOT-23, F.Cu at (100.5, 132.0)
- added Q2: A03401, Package_TO_SOT_SMD:TSOT-23, F.Cu at (141.7, 129.5)
- added Q3: S8050, Package_TO_SOT_SMD:TSOT-23, F.Cu at (148.1, 129.5)
- added Q4: A03401, Package_TO_SOT_SMD:TSOT-23, F.Cu at (151.9, 82.4)
- added Q5: A03401, Package_TO_SOT_SMD:TSOT-23, F.Cu at (156.4, 82.4)
- added R1: NC/0.47R, Resistor_SMD:R_0805_2012Metric, F.Cu at (101.8, 142.2)
- added R10: 10K, Resistor_SMD:R_0805_2012Metric, F.Cu at (106.7, 78.7)
- added R11: 10K, Resistor_SMD:R_0805_2012Metric, F.Cu at (125.1, 58.4)
- added R12: 10K, Resistor_SMD:R_0805_2012Metric, F.Cu at (125.1, 54.6)
- added R13: 0R, Resistor_SMD:R_0805_2012Metric, F.Cu at (135.4, 71.0)
- added R14: 0R, Resistor_SMD:R_0805_2012Metric, F.Cu at (127.8, 71.0)
- added R15: 10K, Resistor_SMD:R_0805_2012Metric, F.Cu at (153.8, 56.4)
- added R16: 200, Resistor_SMD:R_0805_2012Metric, F.Cu at (150.7, 56.4)
- added R17: 20K, Resistor_SMD:R_0805_2012Metric, F.Cu at (150.7, 52.6)
- added R18: 560R, Resistor_SMD:R_0805_2012Metric, F.Cu at (153.8, 52.6)
- added R19: 10K, Resistor_SMD:R_0805_2012Metric, F.Cu at (102.9, 82.5)
- added R2: 3R, Resistor_SMD:R_0805_2012Metric, F.Cu at (99.2, 142.2)
- added R20: 10K, Resistor_SMD:R_0805_2012Metric, F.Cu at (102.9, 72.4)
- added R21: 330R, Resistor_SMD:R_0805_2012Metric, F.Cu at (125.1, 52.1)
- added R22: 0R, Resistor_SMD:R_0805_2012Metric, F.Cu at (154.2, 63.4)
- added R23: NC, Resistor_SMD:R_0805_2012Metric, F.Cu at (153.8, 123.7)
- added R3: 10K, Resistor_SMD:R_0805_2012Metric, F.Cu at (104.0, 126.9)
- added R4: 47K, Resistor_SMD:R_0805_2012Metric, F.Cu at (140.5, 134.5)
- added R5: 10K, Resistor_SMD:R_0805_2012Metric, F.Cu at (145.6, 134.5)
- added R6: NC, Resistor_SMD:R_0805_2012Metric, F.Cu at (147.2, 124.4)
- added R7: 5.1K, Resistor_SMD:R_0805_2012Metric, F.Cu at (155.8, 147.2)
- added R8: 100K, Resistor_SMD:R_0805_2012Metric, F.Cu at (145.6, 137.1)
- added R9: 5.1K, Resistor_SMD:R_0805_2012Metric, F.Cu at (155.8, 144.7)
- added SW1: SW_Push, Button_Switch_SMD:Panasonic_EVQPUL_EVQPUC, F.Cu at (98.6, 68.5)
- added SW2: SW_Push, Button_Switch_SMD:Panasonic_EVQPUL_EVQPUC, F.Cu at (98.6, 78.6)
- added SW3: SW_Push, CustomButtons:KEY-SMD_L4.0-W3.0-LS4.9-1, B.Cu at (150.7, 154.9)
- added SW4: SW_Push, CustomButtons:KEY-SMD_L4.0-W3.0-LS4.9-1, B.Cu at (105.0, 154.9)
- added TP1: AC1, TestPoint:TestPoint_Pad_D3.0mm, F.Cu at (131.6, 71.0)
- added TP2: AC2, TestPoint:TestPoint_Pad_D3.0mm, F.Cu at (124.0, 71.0)
- added U1: BQ51013BRHLR, lcscDownloadLib:VQFN-20_L4.5-W3.5-P0.50-BL-EP_BQ24100RHLR, F.Cu at (143.7, 58.3)
- added U2: XC6220B331MR, Package_TO_SOT_SMD:SOT-23-5, F.Cu at (155.4, 71.6)
- added U3: ESP32-C6-WROOM-1-N8, lcscDownloadLib:WIRELM-SMD_ESP32-C6-WROOM-1, F.Cu at (111.6, 60.3)
- added USB1: TYPE-C 16PIN 2MD, lcscDownloadLib:USB-C-SMD_TYPE-C-16PIN-2MD-073, F.Cu at (150.7, 152.5)
Routing:
- net +3V3: track 0.00 -> 196.8 mm, vias 0 -> 4
- net /Btn1: track 0.00 -> 161.7 mm, vias 0 -> 1
- net /USB_D-: track 0.00 -> 132.4 mm, vias 0 -> 2
- net /USB_D+: track 0.00 -> 132.0 mm, vias 0 -> 2
- net /Btn2: track 0.00 -> 113.9 mm, vias 0 -> 3
- net USB_5V: track 0.00 -> 96.7 mm, vias 0 -> 2
- net /SCREEN_CLK: track 0.00 -> 94.5 mm, vias 0 -> 2
- net +5V: track 0.00 -> 94.3 mm, vias 0 -> 1
- net /SCREEN_CS: track 0.00 -> 94.1 mm, vias 0 -> 2
- net /SCREEN_DIN: track 0.00 -> 93.9 mm, vias 0 -> 2
- net /SCREEN_D/C: track 0.00 -> 92.8 mm, vias 0 -> 2
- net /SCREEN_PWR: track 0.00 -> 91.9 mm, vias 0 -> 2
- net /SCREEN_RST: track 0.00 -> 90.2 mm, vias 0 -> 2
- net /SCREEN_BUSY: track 0.00 -> 88.7 mm, vias 0 -> 2
- net +3.3VP: track 0.00 -> 82.6 mm, vias 0 -> 5
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- added copper zone on B.Cu, net GND
- added copper zone on F.Cu, net GND
Other:
- board outline added: 62.4 x 113.8 mm
- board text added: "+5V"
- board text added: "Boot"
- board text added: "Enable"
- board text added: "GND"

Commit message: still working
Parts:
- turned D4 to 180 degrees
Connections:
- D4 pad 1: Net-(D4-K) -> /MCU_LED
- D4 pad 2: /MCU_LED -> Net-(D4-A)
- R21 pad 2: Net-(D4-K) -> Net-(D4-A)
Routing:
- net GND: track 19.5 -> 30.4 mm
- net Net-(D4-K): track 1.96 -> 0.00 mm
- net Net-(D4-A): track 0.00 -> 1.96 mm
- net /WPT_EN2: track 32.4 -> 31.2 mm
- net Net-(Q4-S): track 7.41 -> 8.34 mm
Changed lines of the file:
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@@
 			(layers "F.Cu" "F.Mask" "F.Paste")
 			(roundrect_rratio 0.243902)
-			(net "Net-(D4-K)")
+			(net "Net-(D4-A)")
 			(pintype "passive")
 		)
@@
 	(footprint "LED_SMD:LED_0805_2012Metric"
 		(layer "F.Cu")
-		(at 128.95 52.07)
+		(at 128.95 52.07 180)
 		(descr "LED SMD 0805 (2012 Metric), square (rectangular) end terminal, IPC-7351 nominal, (Body size source: https://docs.google.com/spreadsheets/d/1BsfQQcO9C6DZCsRaXUlFlo91Tg2WpOkGARC1WS5S8t0/edit?usp=sharing)")
 		(tags "LED")
 		(property "Reference" "D4"
-			(at 0 -1.905 0)
+			(at 0 1.905 0)
 			(layer "F.SilkS")
 			(effects
@@
 		)
 		(property "Sim.Pins" "1=K 2=A"
-			(at 0 0 0)
+			(at 0 0 180)
 			(unlocked yes)
 			(layer "F.Fab")
@@
 		)
 		(property "PARTREV" ""
-			(at 0 0 0)
+			(at 0 0 180)
 			(unlocked yes)
 			(layer "F.Fab")
@@
 		)
 		(property "STANDARD" ""
-			(at 0 0 0)
+			(at 0 0 180)
 			(unlocked yes)
 			(layer "F.Fab")
@@
 		)
 		(property "Sim.Type" ""
-			(at 0 0 0)
+			(at 0 0 180)
 			(unlocked yes)
 			(layer "F.Fab")
@@
 		)
 		(property "LCSC" "C84256"
-			(at 0 0 0)
+			(at 0 0 180)
 			(unlocked yes)
 			(layer "F.Fab")
@@
 		(duplicate_pad_numbers_are_jumpers no)
 		(fp_line
-			(start -1.685 -0.96)
-			(end -1.685 0.96)
+			(start 1 -0.96)
+			(end -1.685 -0.96)
 			(stroke
 				(width 0.12)
@@
 		)
 		(fp_line
-			(start 1 -0.96)
-			(end -1.685 -0.96)
+			(start -1.685 -0.96)
+			(end -1.685 0.96)
 			(stroke
 				(width 0.12)
@@
 		)
 		(fp_line
-			(start -1 -0.3)
-			(end -1 0.6)
+			(start 1 0.6)
+			(end 1 -0.6)
 			(stroke
 				(width 0.1)
@@
 		)
 		(fp_line
-			(start -1 0.6)
-			(end 1 0.6)
+			(start 1 -0.6)
+			(end -0.7 -0.6)
 			(stroke
 				(width 0.1)
@@
 		)
 		(fp_line
-			(start 1 -0.6)
-			(end -0.7 -0.6)
+			(start -1 0.6)
+			(end 1 0.6)
 			(stroke
 				(width 0.1)
@@
 		)
 		(fp_line
-			(start 1 0.6)
-			(end 1 -0.6)
+			(start -1 -0.3)
+			(end -1 0.6)
 			(stroke
 				(width 0.1)
@@
 		)
 		(pad "1" smd roundrect
-			(at -0.9375 0)
+			(at -0.9375 0 180)
 			(size 0.975 1.4)
 			(layers "F.Cu" "F.Mask" "F.Paste")
 			(roundrect_rratio 0.25)
-			(net "Net-(D4-K)")
+			(net "/MCU_LED")
 			(pinfunction "K_1")
 			(pintype "passive")
 		)
 		(pad "2" smd roundrect
-			(at 0.9375 0)
+			(at 0.9375 0 180)
 			(size 0.975 1.4)
 			(layers "F.Cu" "F.Mask" "F.Paste")
 			(roundrect_rratio 0.25)
-			(net "/MCU_LED")
+			(net "Net-(D4-A)")
 			(pinfunction "A_2")
 			(pintype "passive")
@@
 	)
 	(segment
+		(start 147.788308 58.340439)
+		(end 148.59 57.538747)
+		(width 0.2)
+		(layer "F.Cu")
+		(net "GND")
+	)
+	(segment
 		(start 154.440218 150.090877)
 		(end 154.990218 150.640877)
@@
 	)
 	(segment
+		(start 143.685218 58.330877)
+		(end 138.519123 58.330877)
+		(width 0.2)
+		(layer "F.Cu")
+		(net "GND")
+	)
+	(segment
 		(start 147.470218 150.090877)
 		(end 146.900218 150.090877)
@@
 	)
 	(segment
+		(start 143.685218 58.330877)
+		(end 143.69478 58.340439)
+		(width 0.2)
+		(layer "F.Cu")
+		(net "GND")
+	)
+	(segment
+		(start 148.59 57.538747)
+		(end 148.59 57.15)
+		(width 0.2)
+		(layer "F.Cu")
+		(net "GND")
+	)
+	(segment
 		(start 116.100218 127.510877)
 		(end 117.650218 127.510877)
@@
 	)
 	(segment
+		(start 138.519123 58.330877)
+		(end 138.43 58.42)
+		(width 0.2)
+		(layer "F.Cu")
+		(net "GND")
+	)
+	(segment
 		(start 155.435218 69.180877)
 		(end 155.115218 68.860877)
@@
 		(net "GND")
 	)
+	(segment
+		(start 143.69478 58.340439)
+		(end 147.788308 58.340439)
+		(width 0.2)
+		(layer "F.Cu")
+		(net "GND")
+	)
 	(via
 		(at 155.115218 68.860877)
@@
 	)
 	(segment
-		(start 148.130218 58.330877)
-		(end 147.380218 57.580877)
+		(start 147.380218 57.580877)
+		(end 145.935218 57.580877)
 		(width 0.2)
 		(layer "F.Cu")
@@
 	)
 	(segment
-		(start 147.380218 57.580877)
-		(end 145.935218 57.580877)
+		(start 147.539779 57.740439)
+		(end 147.380218 57.580877)
 		(width 0.2)
 		(layer "F.Cu")
@@
 	)
 	(via
-		(at 148.130218 58.330877)
+		(at 147.539779 57.740439)
 		(size 0.6)
 		(drill 0.3)
@@
 	)
 	(segment
-		(start 146.860218 58.330877)
-		(end 148.130218 58.330877)
+		(start 147.539779 57.740439)
+		(end 147.450656 57.740439)
 		(width 0.2)
 		(layer "B.Cu")
@@
 	)
 	(segment
-		(start 124.46 62.23)
+		(start 145.955218 59.235877)
 		(end 127.454123 59.235877)
 		(width 0.2)
@@
 	(segment
 		(start 127.454123 59.235877)
-		(end 145.955218 59.235877)
+		(end 124.46 62.23)
 		(width 0.2)
 		(layer "B.Cu")
@@
 	)
 	(segment
-		(start 145.955218 59.235877)
-		(end 146.860218 58.330877)
+		(start 147.450656 57.740439)
+		(end 145.955218 59.235877)
 		(width 0.2)
 		(layer "B.Cu")
@@
 		(width 0.2)
 		(layer "F.Cu")
-		(net "Net-(D4-K)")
+		(net "Net-(D4-A)")
 	)
 	(segment
@@
 	)
 	(segment
-		(start 150.990218 81.110877)
-		(end 150.990218 82.145877)
-		(width 0.2)
+		(start 156.21 82.55)
+		(end 156.21 81.885659)
+		(width 0.6)
 		(layer "F.Cu")
 		(net "Net-(Q4-S)")
 	)
 	(segment
-		(start 155.750218 81.425877)
-		(end 155.435218 81.110877)
-		(width 0.2)
+		(start 150.990218 81.110877)
+		(end 150.990218 82.410218)
+		(width 0.6)
 		(layer "F.Cu")
 		(net "Net-(Q4-S)")
 	)
 	(segment
-		(start 150.990218 82.145877)
-		(end 151.305218 82.460877)
-		(width 0.2)
+		(start 150.990218 82.410218)
+		(end 151.13 82.55)
+		(width 0.6)
 		(layer "F.Cu")
 		(net "Net-(Q4-S)")
 	)
 	(segment
-		(start 155.750218 82.460877)
-		(end 155.750218 81.425877)
-		(width 0.2)
+		(start 156.21 81.885659)
+		(end 155.435218 81.110877)
+		(width 0.6)
 		(layer "F.Cu")
 		(net "Net-(Q4-S)")
 	)
 	(via
-		(at 155.750218 82.460877)
+		(at 156.21 82.55)
 		(size 0.6)
 		(drill 0.3)
@@
 	)
 	(via
-		(at 151.305218 82.460877)
+		(at 151.13 82.55)
 		(size 0.6)
 		(drill 0.3)
@@
 	)
 	(segment
-		(start 151.305218 82.460877)
-		(end 155.750218 82.460877)
-		(width 0.2)
+		(start 151.13 82.55)
+		(end 156.21 82.55)
+		(width 0.6)
 		(layer "B.Cu")
 		(net "Net-(Q4-S)")

Commit message: fixed card issues
Parts:
- removed AE1: Antenna_Loop, PCB Coils:WPT_COIL
- removed R13, R14: 0R, Resistor_SMD:R_0805_2012Metric
- added R24: 10K, Resistor_SMD:R_0805_2012Metric, F.Cu at (123.4, 62.7)
- added R25: 10K, Resistor_SMD:R_0805_2012Metric, F.Cu at (126.0, 62.7)
- moved C15 1.60 mm to (131.3, 65.3)
Connections:
- C15 pad 1: Net-(C15-Pad1) -> /AC1
- C15 pad 2: Net-(AE1-Pad1) -> /AC2
- C32 pad 1: Net-(AE1-Pad2) -> Net-(C32-Pad1)
- C32 pad 2: Net-(C15-Pad1) -> /AC1
- C33 pad 1: Net-(AE1-Pad2) -> Net-(C32-Pad1)
- C33 pad 2: Net-(C15-Pad1) -> /AC1
- C34 pad 1: Net-(AE1-Pad2) -> Net-(C32-Pad1)
- C34 pad 2: Net-(C15-Pad1) -> /AC1
- TP1 pad 1: /AC1 -> Net-(C32-Pad1)
Routing:
- net Net-(AE1-Pad2): track 35.5 -> 0.00 mm, vias 1 -> 0
- net Net-(C15-Pad1): track 18.6 -> 0.00 mm
- net Net-(AE1-Pad1): track 13.1 -> 0.00 mm
- net Net-(C32-Pad1): track 0.00 -> 12.6 mm
- net /AC1: track 26.2 -> 34.3 mm
- net /AC2: track 41.9 -> 39.8 mm
- net /WPT_EN1: track 33.7 -> 35.7 mm
- net Net-(JP4-A): track 24.7 -> 26.0 mm
- net /WPT_CHG: track 31.7 -> 32.4 mm
- net /WPT_EN2: track 31.2 -> 31.9 mm
